Commit message: Change lidar plugin library

File: urdf/rslidar.urdf.xacro (robot description, xacro)
@@ -46,5 +46,5 @@
       <xacro:unless value="${gpu}">
         <xacro:property name="ray_type" value="ray" />
-        <xacro:property name="plugin_lib" value="libgazebo_ros_velodyne_laser.so" />
+        <xacro:property name="plugin_lib" value="libvelodyne_plugin.so" />
       </xacro:unless>
         <sensor type="${ray_type}" name="${prefix}_sensor">

Commit message: hot fix

File: urdf/rslidar.urdf.xacro (robot description, xacro)
@@ -84,5 +84,5 @@
   </xacro:macro>
   <xacro:macro name="sensor_rslidar_16" params="prefix parent prefix_topic:='lidar_3d' *origin gpu:=false">
-    <xacro:sensor_rslidar prefix="${prefix}" parent="${parent}" prefix_topic="${prefix_topic}" range_min="0.4" range_max="20.0" hfov="180.0" hres="1.0" vfov="20.0" vres="2.0" fps="10.0" gpu="${gpu}" >
+    <xacro:sensor_rslidar prefix="${prefix}" parent="${parent}" prefix_topic="${prefix_topic}" range_min="0.4" range_max="15.0" hfov="100.0" hres="2.0" vfov="18.0" vres="3.0" fps="10.0" gpu="${gpu}" >
       <xacro:insert_block name="origin" />
     </xacro:sensor_rslidar>

File: urdf/teraranger_tr_duo.urdf.xacro (robot description, xacro)
@@ -31,13 +31,13 @@
       <origin xyz="0.02 0 0.012" rpy="0 0 0"/>
 	</joint>
-	<joint name="${prefix}_laser_joint" type="fixed">
+	<!-- <joint name="${prefix}_laser_joint" type="fixed">
       <parent link="${prefix}_base_link"/>
       <child link="${prefix}_laser_link"/>
       <origin xyz="0.02 0 -0.015" rpy="0 0 0"/>
-	</joint>
+	</joint> -->
 	<link name="${prefix}_sonar_link">
 	</link>
-	<link name="${prefix}_laser_link">
-    </link>
+	<!-- <link name="${prefix}_laser_link">
+    </link> -->
 	<!-- TODO add Gazebo stuff for simulation-->
 	<gazebo reference="${prefix}_sonar_link">
@@ -77,5 +77,5 @@
 		</sensor>
 	</gazebo>
-	<gazebo reference="${prefix}_laser_link">
+	<!-- <gazebo reference="${prefix}_laser_link">
 		<material>Gazebo/Yellow</material>
       	<sensor type="ray" name="${prefix}_sensor">
@@ -112,5 +112,5 @@
 			</plugin>
 		</sensor>
-	</gazebo>
+	</gazebo> -->
   </xacro:macro>
 </robot>
